File: PCB_ruche_G2/PCB_ruche_G2.kicad_pcb (KiCad board)
At the start: 2 copper layers, 30 parts, among them J1 RJ12, U1 wisol, U2 STM32L432KC, U3 LDO_jauge, U4 LDO_5_3V3, U6 LDO_DHT, U7 GroveLink, U8 LDO_son, U9 GroveLink

Commit message: Add files via upload
Parts:
- moved Z3 1.27 mm to (245.1, 189.2)
Routing:
- net GND: track 725.2 -> 729.2 mm
- net 3_3V_son: track 108.1 -> 109.4 mm
